File: uv_controler/uv_controler.kicad_pcb (KiCad board)
At the start: 2 copper layers, 28 parts, among them J1 JOY_M, J2 CONTROL_M, J3 CONTROL_D, J4 JOY_D, SW1 RST, U10 FORWARD, U11 BACKWARD, U12 LEFT, U2 DOWN, U3 CAM_UP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

Commit message: arranged pcb roughly
Parts:
- added ?: , , F.Cu at (137.5, 62.0)
- added ?: , , F.Cu at (137.5, 112.0)
- added ?: , , F.Cu at (215.3, 112.0)
- added ?: , , F.Cu at (215.3, 62.0)
- added REF**: MountingHole_3.2mm_M3_DIN965_Pad, MountingHole:MountingHole_3.2mm_M3_DIN965_Pad, F.Cu at (90.5, 62.0)
- added REF**: MountingHole_3.2mm_M3_DIN965_Pad, MountingHole:MountingHole_3.2mm_M3_DIN965_Pad, F.Cu at (215.3, 62.0)
- added REF**: MountingHole_3.2mm_M3_DIN965_Pad, MountingHole:MountingHole_3.2mm_M3_DIN965_Pad, F.Cu at (137.5, 62.0)
- added REF**: MountingHole_3.2mm_M3_DIN965_Pad, MountingHole:MountingHole_3.2mm_M3_DIN965_Pad, F.Cu at (126.5, 112.0)
- added REF**: MountingHole_3.2mm_M3_DIN965_Pad, MountingHole:MountingHole_3.2mm_M3_DIN965_Pad, F.Cu at (30.7, 62.0)
- added REF**: MountingHole_3.2mm_M3_DIN965_Pad, MountingHole:MountingHole_3.2mm_M3_DIN965_Pad, F.Cu at (90.5, 112.0)
- added REF**: MountingHole_3.2mm_M3_DIN965_Pad, MountingHole:MountingHole_3.2mm_M3_DIN965_Pad, F.Cu at (215.3, 112.0)
- added REF**: MountingHole_3.2mm_M3_DIN965_Pad, MountingHole:MountingHole_3.2mm_M3_DIN965_Pad, F.Cu at (101.9, 62.0)
- added REF**: MountingHole_3.2mm_M3_DIN965_Pad, MountingHole:MountingHole_3.2mm_M3_DIN965_Pad, F.Cu at (101.9, 112.0)
- added REF**: MountingHole_3.2mm_M3_DIN965_Pad, MountingHole:MountingHole_3.2mm_M3_DIN965_Pad, F.Cu at (137.5, 112.0)
- added REF**: MountingHole_3.2mm_M3_DIN965_Pad, MountingHole:MountingHole_3.2mm_M3_DIN965_Pad, F.Cu at (126.5, 62.0)
- added REF**: MountingHole_3.2mm_M3_DIN965_Pad, MountingHole:MountingHole_3.2mm_M3_DIN965_Pad, F.Cu at (30.7, 112.0)
- moved R5 61.6 mm to (148.6, 102.9), turned to 180 degrees
- moved U6 61.2 mm to (148.9, 107.4), turned to 180 degrees
- moved R11 57.8 mm to (34.9, 87.0)
- moved U12 57.8 mm to (29.9, 87.0)
- moved J3 51.2 mm to (134.8, 75.8)
- moved R6 49.8 mm to (168.6, 102.9), turned to 180 degrees
- moved R7 49.7 mm to (169.0, 72.9)
- moved U8 49.6 mm to (168.9, 68.1)
- moved U7 49.3 mm to (168.9, 107.4), turned to 180 degrees
- moved R9 46.4 mm to (55.7, 66.2)
- moved U10 46.4 mm to (55.7, 61.2)
- moved J2 46.3 mm to (129.2, 75.8)
- moved SW1 44.9 mm to (116.5, 114.0)
- moved U1 44.8 mm to (107.7, 73.2)
- moved U11 44.3 mm to (55.7, 112.8)
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Connections:
- R10 pad 1: +5VA -> Net-(U11-SUPPLY)
- R11 pad 1: +5VA -> +5VD
- R8 pad 1: +5VA -> +5VD
- R9 pad 1: +5VA -> +5VD
- U10 pad 1: +5VA -> +5VD
- U11 pad 1: +5VA -> Net-(U11-SUPPLY)
- U12 pad 1: +5VA -> +5VD
- U9 pad 1: +5VA -> +5VD
Other:
- board outline added: 194.6 x 60 mm

Commit message: pcb updates, lot of drc errors remain
Parts:
- moved J3 0.96 mm to (135.8, 75.8)
- moved J4 0.94 mm to (92.3, 80.9)
Connections:
- R10 pad 1: Net-(U11-SUPPLY) -> +5VD
- U10 pad 2: GND1 -> GND2
- U11 pad 1: Net-(U11-SUPPLY) -> +5VD
- U11 pad 2: GND1 -> GND2
- U12 pad 2: GND1 -> GND2
- U9 pad 2: GND1 -> GND2
Routing:
- net +5VA: track 0.00 -> 220.7 mm
- net +5VD: track 0.00 -> 147.4 mm
- net /UP_D: track 0.00 -> 90.3 mm
- net /DOWN_D: track 0.00 -> 85.9 mm
- net /CAM_UP_D: track 0.00 -> 75.4 mm
- net /JOY_LEFT_M: track 0.00 -> 75.0 mm
- net /CAM_DOWN_D: track 0.00 -> 63.8 mm
- net /JOY_BACKWARD_D: track 0.00 -> 57.7 mm
- net /SPEED_TOGGLE_D: track 0.00 -> 53.1 mm
- net /JOY_FORWARD_D: track 0.00 -> 46.9 mm
- net /LIGHTS_TOGGLE_D: track 0.00 -> 43.5 mm
- net +5V: track 0.00 -> 38.9 mm
- net Net-(U1-RST): track 0.00 -> 38.3 mm
- net /JOY_RIGHT_D: track 0.00 -> 16.0 mm
- net /UTIL_D: track 0.00 -> 14.7 mm
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- added copper zone on B.Cu, net GND
- added copper zone on F.Cu, net GND
- added copper zone on B.Cu, net GND1
- added copper zone on F.Cu, net GND1
- added copper zone on B.Cu, net GND2
- added copper zone on F.Cu, net GND2

Commit message: pcb cleanup june 6
Parts:
- removed ? (x4): , 
Connections:
- J4 pad 6: /JOY_LEFT_M -> /JOY_LEFT_D
- R11 pad 2: /JOY_LEFT_M -> /JOY_LEFT_D
- U12 pad 3: /JOY_LEFT_M -> /JOY_LEFT_D
Routing:
- net /JOY_LEFT_M: track 75.0 -> 9.57 mm
- net /JOY_LEFT_D: track 0.00 -> 65.4 mm
- net +5VA: track 220.7 -> 243.3 mm
- net /JOY_FORWARD_D: track 46.9 -> 55.2 mm
- net /UTIL_D: track 14.7 -> 19.0 mm
- net +5VD: track 147.4 -> 144.3 mm
- net /JOY_BACKWARD_D: track 57.7 -> 59.2 mm
- net /UP_D: track 90.3 -> 88.9 mm
