File: uv_controler/uv_controler.kicad_sch (KiCad schematic)
At the start: 28 parts, among them J1 JOY_M, J2 CONTROL_M, J3 CONTROL_D, J4 JOY_D, SW1 RST, U10 FORWARD, U11 BACKWARD, U12 LEFT, U2 DOWN, U3 CAM_UP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

Commit message: arranged pcb roughly
Connections:
- net +5VA: no longer R10.1, R11.1, R8.1, R9.1, U10.1 (SUPPLY), U11.1 (SUPPLY), U12.1 (SUPPLY), U9.1 (SUPPLY)
- net +5VD: now also R11.1, R8.1, R9.1, U10.1 (SUPPLY), U12.1 (SUPPLY), U9.1 (SUPPLY)
- new net: R10.1, U11.1 (SUPPLY)
Changed lines of the file:
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@@
 	)
 	(symbol
-		(lib_id "power:+5VA")
-		(at 16.51 123.2929 0)
-		(unit 1)
-		(exclude_from_sim no)
-		(in_bom yes)
-		(on_board yes)
-		(dnp no)
-		(fields_autoplaced yes)
-		(property "Reference" "#PWR030"
-			(at 16.51 127.1029 0)
-			(effects
-				(font
-					(size 1.27 1.27)
-				)
-				(hide yes)
-			)
-		)
-		(property "Value" "+5VA"
-			(at 16.51 118.11 0)
-			(effects
-				(font
-					(size 1.27 1.27)
-				)
-			)
-		)
-		(property "Footprint" ""
-			(at 16.51 123.2929 0)
-			(effects
-				(font
-					(size 1.27 1.27)
-				)
-				(hide yes)
-			)
-		)
-		(property "Datasheet" ""
-			(at 16.51 123.2929 0)
-			(effects
-				(font
-					(size 1.27 1.27)
-				)
-				(hide yes)
-			)
-		)
-		(property "Description" "Power symbol creates a global label with name \"+5VA\""
-			(at 16.51 123.2929 0)
-			(effects
-				(font
-					(size 1.27 1.27)
-				)
-				(hide yes)
-			)
-		)
-		(pin "1"
-		)
-		(instances
-			(project "uv_controler"
-				(path "/9085c9a2-7777-4593-a717-4b341987a03c"
-					(reference "#PWR030")
-					(unit 1)
-				)
-			)
-		)
-	)
-	(symbol
 		(lib_id "power:+5VD")
 		(at 66.04 78.74 0)
@@
 	)
 	(symbol
+		(lib_id "power:+5VD")
+		(at 55.88 63.5 0)
+		(unit 1)
+		(exclude_from_sim no)
+		(in_bom yes)
+		(on_board yes)
+		(dnp no)
+		(fields_autoplaced yes)
+		(property "Reference" "#PWR036"
+			(at 55.88 67.31 0)
+			(effects
+				(font
+					(size 1.27 1.27)
+				)
+				(hide yes)
+			)
+		)
+		(property "Value" "+5VD"
+			(at 55.88 58.42 0)
+			(effects
+				(font
+					(size 1.27 1.27)
+				)
+			)
+		)
+		(property "Footprint" ""
+			(at 55.88 63.5 0)
+			(effects
+				(font
+					(size 1.27 1.27)
+				)
+				(hide yes)
+			)
+		)
+		(property "Datasheet" ""
+			(at 55.88 63.5 0)
+			(effects
+				(font
+					(size 1.27 1.27)
+				)
+				(hide yes)
+			)
+		)
+		(property "Description" "Power symbol creates a global label with name \"+5VD\""
+			(at 55.88 63.5 0)
+			(effects
+				(font
+					(size 1.27 1.27)
+				)
+				(hide yes)
+			)
+		)
+		(pin "1"
+		)
+		(instances
+			(project "uv_controler"
+				(path "/9085c9a2-7777-4593-a717-4b341987a03c"
+					(reference "#PWR036")
+					(unit 1)
+				)
+			)
+		)
+	)
+	(symbol
 		(lib_id "power:GND")
 		(at 147.32 81.28 90)
@@
 	)
 	(symbol
+		(lib_id "power:+5VD")
+		(at 38.1 123.19 0)
+		(unit 1)
+		(exclude_from_sim no)
+		(in_bom yes)
+		(on_board yes)
+		(dnp no)
+		(fields_autoplaced yes)
+		(property "Reference" "#PWR039"
+			(at 38.1 127 0)
+			(effects
+				(font
+					(size 1.27 1.27)
+				)
+				(hide yes)
+			)
+		)
+		(property "Value" "+5VD"
+			(at 38.1 118.11 0)
+			(effects
+				(font
+					(size 1.27 1.27)
+				)
+			)
+		)
+		(property "Footprint" ""
+			(at 38.1 123.19 0)
+			(effects
+				(font
+					(size 1.27 1.27)
+				)
+				(hide yes)
+			)
+		)
+		(property "Datasheet" ""
+			(at 38.1 123.19 0)
+			(effects
+				(font
+					(size 1.27 1.27)
+				)
+				(hide yes)
+			)
+		)
+		(property "Description" "Power symbol creates a global label with name \"+5VD\""
+			(at 38.1 123.19 0)
+			(effects
+				(font
+					(size 1.27 1.27)
+				)
+				(hide yes)
+			)
+		)
+		(pin "1"
+		)
+		(instances
+			(project "uv_controler"
+				(path "/9085c9a2-7777-4593-a717-4b341987a03c"
+					(reference "#PWR039")
+					(unit 1)
+				)
+			)
+		)
+	)
+	(symbol
 		(lib_id "power:GND1")
 		(at 189.23 86.36 90)
@@
 	)
 	(symbol
+		(lib_id "power:+5VD")
+		(at 34.29 64.77 0)
+		(unit 1)
+		(exclude_from_sim no)
+		(in_bom yes)
+		(on_board yes)
+		(dnp no)
+		(fields_autoplaced yes)
+		(property "Reference" "#PWR037"
+			(at 34.29 68.58 0)
+			(effects
+				(font
+					(size 1.27 1.27)
+				)
+				(hide yes)
+			)
+		)
+		(property "Value" "+5VD"
+			(at 34.29 59.69 0)
+			(effects
+				(font
+					(size 1.27 1.27)
+				)
+			)
+		)
+		(property "Footprint" ""
+			(at 34.29 64.77 0)
+			(effects
+				(font
+					(size 1.27 1.27)
+				)
+				(hide yes)
+			)
+		)
+		(property "Datasheet" ""
+			(at 34.29 64.77 0)
+			(effects
+				(font
+					(size 1.27 1.27)
+				)
+				(hide yes)
+			)
+		)
+		(property "Description" "Power symbol creates a global label with name \"+5VD\""
+			(at 34.29 64.77 0)
+			(effects
+				(font
+					(size 1.27 1.27)
+				)
+				(hide yes)
+			)
+		)
+		(pin "1"
+		)
+		(instances
+			(project "uv_controler"
+				(path "/9085c9a2-7777-4593-a717-4b341987a03c"
+					(reference "#PWR037")
+					(unit 1)
+				)
+			)
+		)
+	)
+	(symbol
 		(lib_id "power:+5VA")
 		(at 218.44 71.12 0)
@@
 	)
 	(symbol
-		(lib_id "power:+5VA")
-		(at 34.29 64.77 0)
+		(lib_id "power:+5VD")
+		(at 16.51 123.19 0)
 		(unit 1)
 		(exclude_from_sim no)
@@
 		(dnp no)
 		(fields_autoplaced yes)
-		(property "Reference" "#PWR027"
-			(at 34.29 68.58 0)
+		(property "Reference" "#PWR038"
+			(at 16.51 127 0)
 			(effects
 				(font
@@
 			)
 		)
-		(property "Value" "+5VA"
-			(at 34.29 59.69 0)
+		(property "Value" "+5VD"
+			(at 16.51 118.11 0)
 			(effects
 				(font
@@
 		)
 		(property "Footprint" ""
-			(at 34.29 64.77 0)
+			(at 16.51 123.19 0)
 			(effects
 				(font
@@
 		)
 		(property "Datasheet" ""
-			(at 34.29 64.77 0)
+			(at 16.51 123.19 0)
 			(effects
 				(font
@@
 			)
 		)
-		(property "Description" "Power symbol creates a global label with name \"+5VA\""
-			(at 34.29 64.77 0)
+		(property "Description" "Power symbol creates a global label with name \"+5VD\""
+			(at 16.51 123.19 0)
 			(effects
 				(font
@@
 			(project "uv_controler"
 				(path "/9085c9a2-7777-4593-a717-4b341987a03c"
-					(reference "#PWR027")
+					(reference "#PWR038")
 					(unit 1)
 				)
@@
 	)
 	(symbol
-		(lib_id "power:+5VA")
-		(at 38.1 123.19 0)
-		(unit 1)
-		(exclude_from_sim no)
-		(in_bom yes)
-		(on_board yes)
-		(dnp no)
-		(property "Reference" "#PWR032"
-			(at 38.1 127 0)
-			(effects
-				(font
-					(size 1.27 1.27)
-				)
-				(hide yes)
-			)
-		)
-		(property "Value" "+5VA"
-			(at 38.6513 118.2129 0)
-			(effects
-				(font
-					(size 1.27 1.27)
-				)
-			)
-		)
-		(property "Footprint" ""
-			(at 38.1 123.19 0)
-			(effects
-				(font
-					(size 1.27 1.27)
-				)
-				(hide yes)
-			)
-		)
-		(property "Datasheet" ""
-			(at 38.1 123.19 0)
-			(effects
-				(font
-					(size 1.27 1.27)
-				)
-				(hide yes)
-			)
-		)
-		(property "Description" "Power symbol creates a global label with name \"+5VA\""
-			(at 38.1 123.19 0)
-			(effects
-				(font
-					(size 1.27 1.27)
-				)
-				(hide yes)
-			)
-		)
-		(pin "1"
-		)
-		(instances
-			(project "uv_controler"
-				(path "/9085c9a2-7777-4593-a717-4b341987a03c"
-					(reference "#PWR032")
-					(unit 1)
-				)
-			)
-		)
-	)
-	(symbol
 		(lib_name "SS41F_9")
 		(lib_id "user_symbols:SS41F")
@@
 					(unit 1)
 				)
-			)
-		)
-	)
-	(symbol
-		(lib_id "power:+5VA")
-		(at 55.88 63.5 0)
-		(unit 1)
-		(exclude_from_sim no)
-		(in_bom yes)
-		(on_board yes)
-		(dnp no)
-		(property "Reference" "#PWR029"
-			(at 55.88 67.31 0)
-			(effects
-				(font
-					(size 1.27 1.27)
-				)
-				(hide yes)
-			)
-		)
-		(property "Value" "+5VA"
-			(at 55.88 58.42 0)
-			(effects
-				(font
-					(size 1.27 1.27)
-				)
-			)
-		)
-		(property "Footprint" ""
-			(at 55.88 63.5 0)
-			(effects
-				(font
-					(size 1.27 1.27)
-				)
-				(hide yes)
-			)
-		)
-		(property "Datasheet" ""
-			(at 55.88 63.5 0)
-			(effects
-				(font
-					(size 1.27 1.27)
-				)
-				(hide yes)
-			)
-		)
-		(property "Description" "Power symbol creates a global label with name \"+5VA\""
-			(at 55.88 63.5 0)
-			(effects
-				(font
-					(size 1.27 1.27)
-				)
-				(hide yes)
-			)
-		)
-		(pin "1"
-		)
-		(instances
-			(project "uv_controler"
-				(path "/9085c9a2-7777-4593-a717-4b341987a03c"
-					(reference "#PWR029")
-					(unit 1)
-				)

Commit message: pcb updates, lot of drc errors remain
Connections:
- net +5VD: now also R10.1, U11.1 (SUPPLY)
- net GND1: no longer U10.2 (GND), U11.2 (GND), U12.2 (GND), U9.2 (GND)
- net GND2: now also U10.2 (GND), U11.2 (GND), U12.2 (GND), U9.2 (GND)

Commit message: pcb cleanup june 6
Connections:
- net JOY_LEFT_M: no longer J4.6 (Pin_6), R11.2, U12.3 (OUTPUT)
- new net JOY_LEFT_D: J4.6 (Pin_6), R11.2, U12.3 (OUTPUT)
Changed lines of the file:
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@@
 		)
 	)
-	(label "JOY_LEFT_M"
+	(label "JOY_LEFT_D"
 		(at 50.8 96.52 0)
 		(effects
